Commit message: Added fix for hydroshear_med

File: odyssey/urdf/med_calib_hydroshear.urdf (robot description, URDF)
Before this commit: robot iiwa, 13 links, 11 joints
Joints:
- removed joint mount_joint
- added joint ee_mount_joint: type fixed, parent iiwa_link_ee_kuka, child indenter_mount, origin xyz=0 0 0.0 rpy=0 0 0
- added joint mount_sphere_joint: type fixed, parent indenter_mount, child indenter_sphere, origin xyz=0 0 0.01969 rpy=0 0 0
