Commit message: Added sphere and indenter_mount into med calibration urdf.

File: odyssey/urdf/gs_mini_hydroshear_calib.urdf (robot description, URDF)
Before this commit: robot gelsight_mini_calibration, 2 links, 1 joints
Links:
- added link gelpad; collision mesh filename=./gelsight_mini/gsmini_elastomer_transformed.obj; visual mesh filename=./gelsight_mini/gsmini_elastomer_transformed.obj
- added link mount; collision mesh filename=./calib_assets/gelsight_mount/gelsight_mount.obj; visual mesh filename=./calib_assets/gelsight_mount/gelsight_mount.obj
- link base: geometry 
Joints:
- added joint base_joint: type fixed, parent base, child mount, origin xyz=0 0 0 rpy=0 0 0
- added joint gelpad_shell_fixed: type fixed, parent gelsight_shell, child gelpad, origin xyz=0 0 0.00 rpy=0 0 0

File: odyssey/urdf/med_calib_hydroshear.urdf (robot description, URDF)
Before this commit: robot iiwa, 11 links, 10 joints
Links:
- added link indenter_mount; collision mesh filename=./calib_assets/indenter_mount/indenter_mount.obj; visual mesh filename=./calib_assets/indenter_mount/indenter_mount.obj
- added link indenter_sphere; collision mesh filename=./calib_assets/24mm_sphere/24mm_sphere.obj; visual mesh filename=./calib_assets/24mm_sphere/24mm_sphere.obj
Joints:
- added joint mount_joint: type fixed, parent indenter_mount, child indenter_sphere, origin xyz=0 0 0.012 rpy=0 0 0

Commit message: Added 35mm sphere for real-world and fixed urdf of kuka to not have gap between iiwa_link_0 and iiwa_link_1

File: odyssey/urdf/gs_mini_hydroshear_calib.urdf (robot description, URDF)
Before this commit: robot gelsight_mini_calibration, 4 links, 3 joints
Joints:
- joint shell_base_fixed: origin xyz=0.713041081 0 0.0060 rpy=0 0 0 -> xyz=0.713041081 0 0.0060 rpy=0 0 1.57079633; parent base -> mount

File: odyssey/urdf/med_calib_hydroshear.urdf (robot description, URDF)
Before this commit: robot iiwa, 13 links, 11 joints
Links:
- link indenter_sphere: geometry collision mesh filename=./calib_assets/35mm_sphere/35mm_sphere.obj; visual mesh filename=./calib_assets/35mm_sphere/35mm_sphere.obj
Joints:
- joint iiwa_joint_1: origin xyz=0 0 0.1575 rpy=0 0 0 -> xyz=0.0 0.0 0.147 rpy=0 0 0

Commit message: Updated .urdf files for calibration to match real world calib (and cross-referencing with hydroshear repo).

File: odyssey/urdf/gs_mini_hydroshear_calib.urdf (robot description, URDF)
Before this commit: robot gelsight_mini_calibration, 4 links, 3 joints
Links:
- link gelpad: geometry collision mesh filename=./gelsight_mini/gsmini_elastomer_transformed_enclosed.obj; visual mesh filename=./gelsight_mini/gsmini_elastomer_transformed_enclosed.obj

File: odyssey/urdf/med_calib_hydroshear.urdf (robot description, URDF)
Before this commit: robot iiwa, 13 links, 12 joints
Joints:
- joint mount_sphere_joint: origin xyz=0 0 0.01969 rpy=0 0 0 -> xyz=0 0 0.0196969 rpy=0 0 0

Commit message: Want yellow color to be in visual when using gsmini hydroshear calibration urdf

File: odyssey/urdf/gs_mini_hydroshear_calib.urdf (robot description, URDF)
Before this commit: robot gelsight_mini_calibration, 4 links, 3 joints
Links:
- link gelpad: geometry collision mesh filename=./gelsight_mini/gsmini_elastomer_transformed_enclosed.obj; visual mesh filename=./gelsight_mini/gsmini_elastomer_transformed.obj
